File: cpNode-IOX.kicad_sch (KiCad schematic)
At the start: 0 parts

Commit message: chore(spike1): checkpoint metadata normalization and ERC fixes
Parts:
- added C1: 220uF, SPCoast:CP_Elec_8x10, symbol Device:C_Polarized_US
- added C2: 0.1uF, SPCoast:0603-CAP, symbol SPCoast:C
- added C3: 1uF, SPCoast:0603-CAP, symbol SPCoast:C
- added D1: BAT54A, Package_TO_SOT_SMD:SOT-23, symbol Diode:BAT54A
- added J1: DCJ0202, Connector_BarrelJack:BarrelJack_Kycon_KLDX-0202-xC_Horizontal, symbol SPCoast:Conn_DC-POWER
- added J2: Vin, Connector_PinHeader_2.54mm:PinHeader_1x04_P2.54mm_Vertical, symbol SPCoast:Conn_01x04
- added J3: Vout, Connector_PinHeader_2.54mm:PinHeader_1x04_P2.54mm_Vertical, symbol SPCoast:Conn_01x04
- added LED1: Green, SPCoast:0603-LED, symbol SPCoast:LED
- added LED2: Red, SPCoast:0603-LED, symbol SPCoast:LED
- added PWR-LABEL1: ${V} @${A}, SPCoast:SILK_Label-Power_CP, symbol SPCoast:DOC_Label-Power_CP
- added Q1: Q_P-FET_8A_SOP-8_A04443, Package_SO:HTSOP-8-1EP_3.9x4.9mm_P1.27mm_EP2.4x3.2mm, symbol SPCoast:MOSFET-P_AO4443
- added R35, R36: 4k7, SPCoast:0603-RES, symbol SPCoast:R
- added VR1: LM78M05_TO252-2, Package_TO_SOT_SMD:TO-252-2, symbol Regulator_Linear:LM78M05_TO252
Connections:
- new net: C1.1, C2.1, Q1.1 (S), Q1.2 (S), Q1.3 (S), VR1.1 (VI)
- new net: LED1.1 (K), R35.1
- new net: D1.3, LED2.1 (K), R36.1
- new net +5V: C3.1, LED1.2 (A), VR1.3 (VO)
- new net +VDC: J1.1, J2.2 (Pin_2), J2.3 (Pin_3), J3.2 (Pin_2), J3.3 (Pin_3), Q1.5 (D), Q1.6 (D), Q1.7 (D), Q1.8 (D), Q1.9 (D), R36.2
- new net GND: C1.2, C2.2, C3.2, D1.2, J1.2, J1.3, J2.1 (Pin_1), J2.4 (Pin_4), J3.1 (Pin_1), J3.4 (Pin_4), LED2.2 (A), Q1.4 (G), R35.2, VR1.2 (GND)
- no-connect marks 0 -> 1
Other:
- note added: "Power Good"
- note added: "Power Reversed"
- note added: "Power Supply"
- note added: "Reverse Voltage Protection (Max Vgs=+/-20v, no zener needed)"
- company: (none) -> SPCoast
- title: (none) -> cpNode-IOX

Commit message: chore(spike1): step-03 exit - sync design block + fixes from broken sandbox
Per the corrected step lifecycle: -broken's content (design block +
step-2 debt retired via symbol restore/PWR_FLAG/metadata fixes) is
copied here as the clean exit state, since step 3 introduced zero new
defects (design-block checks were clean from the start). This repo is
the sandbox where kDoctor fixers actually run; -broken is left
untouched as the permanent before-state.

Result: design-block/ERC/metadata checks all findings=0.
Parts:
- renumbered R35 to R1, R36 to R2

Commit message: Step-04 complete: all ERC violations fixed, sandbox clean
- Re-annotated schematic (cleared duplicate refdes J12/J13, unannotated J_{I2C-IN}?)
- Updated symbols from library (cleared 22 lib_symbol_mismatch warnings)
- Converted SCL/SDA local labels → global (cleared 2 same_local_global_label warnings)
- Fixed footprint references (preparation for Step-05 PCB work)
- Manually rewired power connector after I2C block library update (wire detachment issue)
- Final state: 0 ERC errors, 0 warnings (completely clean)
- ERC.rpt timestamp: 2026-07-21T21:03:47
- Validation: poc/erc_drc_summary.py reports total: 0
Parts:
- added Board1: (no value), SPCoast:Board_068x80, symbol SPCoast:Board
- added DOC1: ${TITLE}, SPCoast:SILK_BoardID, symbol SPCoast:DOC_Label-Board
- added J1, J11, J12, J15, J16, J2: CON_1x04-0.100-screw, Connector_PinHeader_2.54mm:PinHeader_1x04_P2.54mm_Vertical, symbol SPCoast:Conn_01x04
- added J10, J19, J3, J7, J8, J9: Conn_01x02, Connector_PinHeader_2.54mm:PinHeader_1x02_P2.54mm_Vertical, symbol SPCoast:Conn_01x02
- added J13, J14, J17, J18: Conn_01x08, Connector_PinHeader_2.54mm:PinHeader_1x08_P2.54mm_Vertical, symbol SPCoast:Conn_01x08
- added J_{I2C-IN}1: I2C, SPCoast:Connector_I2C-0.100_R, symbol SPCoast:Conn_I2C
- added J_{I2C-OUT}1: I2C, SPCoast:Connector_I2C-0.100_L, symbol SPCoast:Conn_I2C
- added R1, R2: 2k2, SPCoast:0603-RES, symbol SPCoast:R
- added R10, R11, R12, R13, R14, R8, R9: 220R, SPCoast:0603-RES, symbol SPCoast:R
- added R5, R6, R7: 10k0, SPCoast:0603-RES, symbol SPCoast:R
- added SJ1, SJ10, SJ11, SJ12, SJ13, SJ14, SJ15, SJ16, SJ2, SJ3, SJ4, SJ5, SJ6, SJ7, SJ8, SJ9: OFF, Jumper:SolderJumper-2_P1.3mm_Bridged_RoundedPad1.0x1.5mm, symbol Jumper:SolderJumper_2_Bridged
- added SW1: (no value), SPCoast:SW-EDG-04, symbol SPCoast:SW_EDG-04
- added U1: MCP23017_SO, Package_SO:SOIC-28W_7.5x17.9mm_P1.27mm, symbol SPCoast:MCP23017_SO
- added U2: 74HC4511D,653, Package_SO:SOIC-16_3.9x9.9mm_P1.27mm, symbol 4xxx_IEEE:4511
- added U3: ARKLED SM420561N, Display_7Segment:D1X8K, symbol Display_Character:D1X8K-14BL
- renumbered J2 to J4, J3 to J5, J1 to J6, R1 to R3, R2 to R4
Connections:
- net +5V: now also J1.1 (Pin_1), J1.2 (Pin_2), J1.3 (Pin_3), J1.4 (Pin_4), J10.1 (Pin_1), J19.1 (Pin_1), J3.1 (Pin_1), J7.1 (Pin_1), J_{I2C-OUT}1.2, R1.1, R2.1, R5.1, R6.1, R7.1, U1.18 (~{RESET}), U1.9 (VDD), U2.16 (Vdd), U2.3 (~{LT}), U2.4 (~{BI})
- net GND: now also J10.2 (Pin_2), J19.2 (Pin_2), J2.1 (Pin_1), J2.2 (Pin_2), J2.3 (Pin_3), J2.4 (Pin_4), J3.2 (Pin_2), J7.2 (Pin_2), J_{I2C-IN}1.1, J_{I2C-OUT}1.1, SW1.2, SW1.3, SW1.4, U1.10 (VSS), U2.5 (~{EL}), U2.6 (DD), U2.8 (Vss), U3.3 (CC), U3.5 (DP), U3.8 (CC)
- new net: J9.1 (Pin_1), R2.2
- new net: J16.4 (Pin_4), J17.1 (Pin_1), SJ16.1 (A)
- new net: J11.2 (Pin_2), J13.7 (Pin_7), SJ2.1 (A)
- new net: J14.7 (Pin_7), SJ2.2 (B), U1.2 (GPB1)
- new net: J16.3 (Pin_3), J17.2 (Pin_2), SJ15.1 (A)
- new net: J12.1 (Pin_1), J13.4 (Pin_4), SJ5.1 (A)
- new net: J12.2 (Pin_2), J13.3 (Pin_3), SJ6.1 (A)
- new net: J12.3 (Pin_3), J13.2 (Pin_2), SJ7.1 (A)
- new net: J12.4 (Pin_4), J13.1 (Pin_1), SJ8.1 (A)
- new net: J16.1 (Pin_1), J17.4 (Pin_4), SJ13.1 (A)
- new net: J16.2 (Pin_2), J17.3 (Pin_3), SJ14.1 (A)
- new net: R9.1, U2.12 (Qb)
- new net: R9.2, U3.6 (B)
- new net: R12.1, U2.9 (Qe)
- new net: R12.2, U3.1 (E)
- new net: J15.4 (Pin_4), J17.5 (Pin_5), SJ12.1 (A)
- new net: J15.3 (Pin_3), J17.6 (Pin_6), SJ11.1 (A)
- new net: J15.2 (Pin_2), J17.7 (Pin_7), SJ10.1 (A)
- new net: J15.1 (Pin_1), J17.8 (Pin_8), SJ9.1 (A)
- new net: J14.1 (Pin_1), SJ8.2 (B), U1.8 (GPB7)
- new net: J14.2 (Pin_2), SJ7.2 (B), U1.7 (GPB6)
- new net: J14.3 (Pin_3), SJ6.2 (B), U1.6 (GPB5)
- new net: J14.4 (Pin_4), SJ5.2 (B), U1.5 (GPB4)
- new net: J14.5 (Pin_5), SJ4.2 (B), U1.4 (GPB3)
- new net: J14.6 (Pin_6), SJ3.2 (B), U1.3 (GPB2)
- new net: J14.8 (Pin_8), SJ1.2 (B), U1.1 (GPB0)
- new net: R14.1, U2.14 (Qg)
- new net: R14.2, U3.10 (G)
- new net: J11.1 (Pin_1), J13.8 (Pin_8), SJ1.1 (A)
- new net: J11.3 (Pin_3), J13.6 (Pin_6), SJ3.1 (A)
- new net: J11.4 (Pin_4), J13.5 (Pin_5), SJ4.1 (A)
- new net: R8.1, U2.13 (Qa)
- new net: R8.2, U3.7 (A)
- new net: J8.1 (Pin_1), R1.2
- new net: R11.1, U2.10 (Qd)
- new net: R11.2, U3.2 (D)
- new net: R10.1, U2.11 (Qc)
- new net: R13.1, U2.15 (Qf)
- new net: R10.2, U3.4 (C)
- new net: R13.2, U3.9 (F)
- new net A0: R7.2, SW1.5, U1.15 (A0), U2.7 (DA)
- new net A1: R6.2, SW1.6, U1.16 (A1), U2.1 (DB)
- new net A2: R5.2, SW1.7, U1.17 (A2), U2.2 (DC)
- new net GPA0: J18.1 (Pin_1), SJ16.2 (B), U1.28 (GPA7)
- new net GPA1: J18.2 (Pin_2), SJ15.2 (B), U1.27 (GPA6)
- new net GPA2: J18.3 (Pin_3), SJ14.2 (B), U1.26 (GPA5)
- new net GPA3: J18.4 (Pin_4), SJ13.2 (B), U1.25 (GPA4)
- new net GPA4: J18.5 (Pin_5), SJ12.2 (B), U1.24 (GPA3)
- new net GPA5: J18.6 (Pin_6), SJ11.2 (B), U1.23 (GPA2)
- new net GPA6: J18.7 (Pin_7), SJ10.2 (B), U1.22 (GPA1)
- new net GPA7: J18.8 (Pin_8), SJ9.2 (B), U1.21 (GPA0)
- new net SCL: J8.2 (Pin_2), J_{I2C-IN}1.4, J_{I2C-OUT}1.4, U1.12 (SCK)
- new net SDA: J9.2 (Pin_2), J_{I2C-IN}1.3, J_{I2C-OUT}1.3, U1.13 (SDA)
- no-connect marks 1 -> 6
Other:
- note added: "I2C"
- note added: "I2C Termination"
- note added: "IOX Plugin Footprint"
