File: cpNode-IOX.kicad_sch (KiCad schematic)
At the start: 66 parts, among them J1 CON_1x04-0.100-screw, J10 Conn_01x02, J11 CON_1x04-0.100-screw, J12 CON_1x04-0.100-screw, J13 Conn_01x08, J14 Conn_01x08, J15 CON_1x04-0.100-screw, J16 CON_1x04-0.100-screw, J17 Conn_01x08, J18 Conn_01x08, J19 Conn_01x02, J2 CON_1x04-0.100-screw, J3 Conn_01x02, J4 Vin, J5 Vout, J6 DCJ0202, J7 Conn_01x02, J8 Conn_01x02, J9 Conn_01x02, Q1 Q_P-FET_8A_SOP-8_A04443, U1 MCP23017_SO, U2 74HC4511D,653, U3 ARKLED SM420561N

Commit message: pcb+sch: Step-05 PCB layout complete, ported from cpNode-IOX-broken
Ports the entire Step-05 PCB-layout effort from cpNode-IOX-broken into
this sandbox in one shot, per the standing "designer-work happens in
broken, gets copied to clean" workflow -- this copy was deferred across
the whole step instead of happening incrementally, so it lands as a
single large diff rather than per-checkpoint.

What this brings in:
- Full PCB layout: netlist import, placement, routing (0 unconnected
  items, 0 schematic parity issues), 3 DRC findings excluded with a
  documented rationale (courtyards_overlap x1, pth_inside_courtyard x2
  -- Tyco mounting-track clearance, see FIELD-NOTES.md).
- Silkscreen text and layout polish.
- Metadata fixes: Comment9 typo (schematic/pcb title-block agreement),
  Comment2 (summary) sch/pcb agreement, schematic/pcb revision fields.
- SPCoast-eagle:+5V remapped off the legacy Eagle-import symbol.
- SPCoast footprint-library housekeeping reflected on the placed
  instances (Board1/SILK_BoardID/SILK_Label-Power_CP/SolderJumper-2
  attribute sync with their (separately updated) library masters).
- Embedded .kicad_wks re-synced to the current canonical template.

Verified via the full kDoctor check suite against this file set before
committing: ERC 0, DRC 0 active/unconnected/parity (3 excluded with
rationale), metadata 0, symbol lineage 0, footprint-library drift 0,
embedded-wks drift 0 (matches_canonical), design blocks 0/0.

This supersedes cpNode-IOX's own prior, independent issues (stale
Board_068x80 footprint reference with a zero-pad mismatch, unremapped
SPCoast-eagle:+5V, missing revision fields) as a side effect of the
wholesale copy, not via a separate fix pass.

Co-Authored-By: Oz <oz-agent@warp.dev>
Parts:
- Board1: footprint SPCoast:Board_068x80 -> SPCoast:Board_068x110
- PWR-LABEL1: now left out of the parts list
Connections:
- net at J16.4 (Pin_4), SJ16.1 (A): now also J17.8 (Pin_8); no longer J17.1 (Pin_1)
- net at J11.2 (Pin_2), SJ2.1 (A): now also J13.2 (Pin_2); no longer J13.7 (Pin_7)
- net at SJ2.2 (B), U1.2 (GPB1): now also J14.2 (Pin_2); no longer J14.7 (Pin_7)
- net at J16.3 (Pin_3), SJ15.1 (A): now also J17.7 (Pin_7); no longer J17.2 (Pin_2)
- net at J12.1 (Pin_1), SJ5.1 (A): now also J13.5 (Pin_5); no longer J13.4 (Pin_4)
- net at J12.2 (Pin_2), SJ6.1 (A): now also J13.6 (Pin_6); no longer J13.3 (Pin_3)
- net at J12.3 (Pin_3), SJ7.1 (A): now also J13.7 (Pin_7); no longer J13.2 (Pin_2)
- net at J12.4 (Pin_4), SJ8.1 (A): now also J13.8 (Pin_8); no longer J13.1 (Pin_1)
- net at J16.1 (Pin_1), SJ13.1 (A): now also J17.5 (Pin_5); no longer J17.4 (Pin_4)
- net at J16.2 (Pin_2), SJ14.1 (A): now also J17.6 (Pin_6); no longer J17.3 (Pin_3)
- net at J15.4 (Pin_4), SJ12.1 (A): now also J17.4 (Pin_4); no longer J17.5 (Pin_5)
- net at J15.3 (Pin_3), SJ11.1 (A): now also J17.3 (Pin_3); no longer J17.6 (Pin_6)
- net at J15.2 (Pin_2), SJ10.1 (A): now also J17.2 (Pin_2); no longer J17.7 (Pin_7)
- net at J15.1 (Pin_1), SJ9.1 (A): now also J17.1 (Pin_1); no longer J17.8 (Pin_8)
- net at SJ8.2 (B), U1.8 (GPB7): now also J14.8 (Pin_8); no longer J14.1 (Pin_1)
- net at SJ7.2 (B), U1.7 (GPB6): now also J14.7 (Pin_7); no longer J14.2 (Pin_2)
- net at SJ6.2 (B), U1.6 (GPB5): now also J14.6 (Pin_6); no longer J14.3 (Pin_3)
- net at SJ5.2 (B), U1.5 (GPB4): now also J14.5 (Pin_5); no longer J14.4 (Pin_4)
- net at SJ4.2 (B), U1.4 (GPB3): now also J14.4 (Pin_4); no longer J14.5 (Pin_5)
- net at SJ3.2 (B), U1.3 (GPB2): now also J14.3 (Pin_3); no longer J14.6 (Pin_6)
- net at SJ1.2 (B), U1.1 (GPB0): now also J14.1 (Pin_1); no longer J14.8 (Pin_8)
- net at J11.1 (Pin_1), SJ1.1 (A): now also J13.1 (Pin_1); no longer J13.8 (Pin_8)
- net at J11.3 (Pin_3), SJ3.1 (A): now also J13.3 (Pin_3); no longer J13.6 (Pin_6)
- net at J11.4 (Pin_4), SJ4.1 (A): now also J13.4 (Pin_4); no longer J13.5 (Pin_5)
- net GPA0: no longer names the net of SJ16.2 (B), U1.28 (GPA7)
- net GPA0: now also J18.8 (Pin_8); no longer J18.1 (Pin_1)
- net GPA1: no longer names the net of SJ15.2 (B), U1.27 (GPA6)
- net GPA1: now also J18.7 (Pin_7); no longer J18.2 (Pin_2)
- net GPA2: no longer names the net of SJ14.2 (B), U1.26 (GPA5)
- net GPA2: now also J18.6 (Pin_6); no longer J18.3 (Pin_3)
- net GPA3: no longer names the net of SJ13.2 (B), U1.25 (GPA4)
- net GPA3: now also J18.5 (Pin_5); no longer J18.4 (Pin_4)
- net GPA4: no longer names the net of SJ12.2 (B), U1.24 (GPA3)
- net GPA4: now also J18.4 (Pin_4); no longer J18.5 (Pin_5)
- net GPA5: no longer names the net of SJ11.2 (B), U1.23 (GPA2)
- net GPA5: now also J18.3 (Pin_3); no longer J18.6 (Pin_6)
- net GPA6: no longer names the net of SJ10.2 (B), U1.22 (GPA1)
- net GPA6: now also J18.2 (Pin_2); no longer J18.7 (Pin_7)
- net GPA7: no longer names the net of SJ9.2 (B), U1.21 (GPA0)
- net GPA7: now also J18.1 (Pin_1); no longer J18.8 (Pin_8)

Commit message: moved screw connectors
Parts:
- U2: value 74HC4511D,653 -> IC_SOIC-16_74HC4511; LCSC C87661 -> (none)
Changed lines of the file:
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@@
 			)
 		)
-		(property "Value" "74HC4511D,653"
+		(property "Value" "IC_SOIC-16_74HC4511"
 			(at 198.9933 93.98 0)
 			(show_name no)
@@
 			(at 196.85 106.68 0)
 			(hide yes)
-			(show_name no)
-			(do_not_autoplace no)
-			(effects
-				(font
-					(size 1.27 1.27)
-				)
-			)
-		)
-		(property "LCSC" "C87661"
-			(at 196.85 106.68 0)
-			(hide yes)
