File: cpNode-IOX.kicad_pcb (KiCad board)
At the start: 0 parts

Commit message: pcb+sch: Step-05 PCB layout complete, ported from cpNode-IOX-broken
Ports the entire Step-05 PCB-layout effort from cpNode-IOX-broken into
this sandbox in one shot, per the standing "designer-work happens in
broken, gets copied to clean" workflow -- this copy was deferred across
the whole step instead of happening incrementally, so it lands as a
single large diff rather than per-checkpoint.

What this brings in:
- Full PCB layout: netlist import, placement, routing (0 unconnected
  items, 0 schematic parity issues), 3 DRC findings excluded with a
  documented rationale (courtyards_overlap x1, pth_inside_courtyard x2
  -- Tyco mounting-track clearance, see FIELD-NOTES.md).
- Silkscreen text and layout polish.
- Metadata fixes: Comment9 typo (schematic/pcb title-block agreement),
  Comment2 (summary) sch/pcb agreement, schematic/pcb revision fields.
- SPCoast-eagle:+5V remapped off the legacy Eagle-import symbol.
- SPCoast footprint-library housekeeping reflected on the placed
  instances (Board1/SILK_BoardID/SILK_Label-Power_CP/SolderJumper-2
  attribute sync with their (separately updated) library masters).
- Embedded .kicad_wks re-synced to the current canonical template.

Verified via the full kDoctor check suite against this file set before
committing: ERC 0, DRC 0 active/unconnected/parity (3 excluded with
rationale), metadata 0, symbol lineage 0, footprint-library drift 0,
embedded-wks drift 0 (matches_canonical), design blocks 0/0.

This supersedes cpNode-IOX's own prior, independent issues (stale
Board_068x80 footprint reference with a zero-pad mismatch, unremapped
SPCoast-eagle:+5V, missing revision fields) as a side effect of the
wholesale copy, not via a separate fix pass.

Co-Authored-By: Oz <oz-agent@warp.dev>
Parts:
- added Board1: ~, SPCoast:Board_068x110, F.Cu at (127.0, 127.0)
- added C1: 220uF, SPCoast:CP_Elec_8x10, F.Cu at (153.0, 89.5)
- added C2: 0.1uF, SPCoast:0603-CAP, F.Cu at (156.2, 81.3)
- added C3: 1uF, SPCoast:0603-CAP, F.Cu at (156.2, 77.5)
- added D1: BAT54A, Package_TO_SOT_SMD:SOT-23, F.Cu at (139.4, 114.9)
- added DOC1: cpNode-IOX, SPCoast:SILK_BoardID, F.Cu at (204.8, 123.1)
- added J1: CON_1x04-0.100-screw, Connector_PinHeader_2.54mm:PinHeader_1x04_P2.54mm_Vertical, F.Cu at (139.1, 66.0)
- added J10: Conn_01x02, Connector_PinHeader_2.54mm:PinHeader_1x02_P2.54mm_Vertical, F.Cu at (191.8, 81.3)
- added J11: CON_1x04-0.100-screw, Connector_PinHeader_2.54mm:PinHeader_1x04_P2.54mm_Vertical, F.Cu at (188.6, 66.0)
- added J12: CON_1x04-0.100-screw, Connector_PinHeader_2.54mm:PinHeader_1x04_P2.54mm_Vertical, F.Cu at (175.3, 66.1)
- added J13: Conn_01x08, Connector_PinHeader_2.54mm:PinHeader_1x08_P2.54mm_Vertical, F.Cu at (186.7, 71.1)
- added J14: Conn_01x08, Connector_PinHeader_2.54mm:PinHeader_1x08_P2.54mm_Vertical, F.Cu at (186.7, 81.3)
- added J15: CON_1x04-0.100-screw, Connector_PinHeader_2.54mm:PinHeader_1x04_P2.54mm_Vertical, F.Cu at (224.2, 66.8)
- added J16: CON_1x04-0.100-screw, Connector_PinHeader_2.54mm:PinHeader_1x04_P2.54mm_Vertical, F.Cu at (211.5, 66.8)
- added J17: Conn_01x08, Connector_PinHeader_2.54mm:PinHeader_1x08_P2.54mm_Vertical, F.Cu at (222.9, 71.1)
- added J18: Conn_01x08, Connector_PinHeader_2.54mm:PinHeader_1x08_P2.54mm_Vertical, F.Cu at (222.9, 81.3)
- added J19: Conn_01x02, Connector_PinHeader_2.54mm:PinHeader_1x02_P2.54mm_Vertical, F.Cu at (227.9, 81.3)
- added J2: CON_1x04-0.100-screw, Connector_PinHeader_2.54mm:PinHeader_1x04_P2.54mm_Vertical, F.Cu at (151.8, 66.0)
- added J3: Conn_01x02, Connector_PinHeader_2.54mm:PinHeader_1x02_P2.54mm_Vertical, F.Cu at (156.2, 73.7)
- added J4: Vin, Connector_PinHeader_2.54mm:PinHeader_1x04_P2.54mm_Vertical, F.Cu at (132.1, 106.0)
- added J5: Vout, Connector_PinHeader_2.54mm:PinHeader_1x04_P2.54mm_Vertical, F.Cu at (232.4, 106.7)
- added J6: DCJ0202, Connector_BarrelJack:BarrelJack_Kycon_KLDX-0202-xC_Horizontal, F.Cu at (158.1, 116.9)
- added J7: Conn_01x02, Connector_PinHeader_2.54mm:PinHeader_1x02_P2.54mm_Vertical, F.Cu at (156.2, 69.8)
- added J8: Conn_01x02, Connector_PinHeader_2.54mm:PinHeader_1x02_P2.54mm_Vertical, F.Cu at (139.9, 97.8)
- added J9: Conn_01x02, Connector_PinHeader_2.54mm:PinHeader_1x02_P2.54mm_Vertical, F.Cu at (144.5, 97.8)
- added J_{I2C-IN}1: I2C, SPCoast:Connector_I2C-0.100_R, F.Cu at (132.1, 99.7)
- added J_{I2C-OUT}1: I2C, SPCoast:Connector_I2C-0.100_L, F.Cu at (232.4, 100.3)
- added LED1: Green, SPCoast:0603-LED, F.Cu at (146.1, 118.7)
- added LED2: Red, SPCoast:0603-LED, F.Cu at (142.2, 118.7)
- added PWR-LABEL1: 12VDC @1A, SPCoast:SILK_Label-Power_CP, F.Cu at (168.1, 118.5)
- added Q1: Q_P-FET_8A_SOP-8_A04443, Package_SO:HTSOP-8-1EP_3.9x4.9mm_P1.27mm_EP2.4x3.2mm, F.Cu at (159.4, 98.4)
- added R1: 2k2, SPCoast:0603-RES, F.Cu at (139.7, 92.7)
- added R10: 220R, SPCoast:0603-RES, F.Cu at (203.8, 104.0)
- added R11: 220R, SPCoast:0603-RES, F.Cu at (203.8, 105.9)
- added R12: 220R, SPCoast:0603-RES, F.Cu at (203.8, 107.8)
- added R13: 220R, SPCoast:0603-RES, F.Cu at (203.8, 96.4)
- added R14: 220R, SPCoast:0603-RES, F.Cu at (203.8, 98.3)
- added R2: 2k2, SPCoast:0603-RES, F.Cu at (144.1, 92.7)
- added R3: 4k7, SPCoast:0603-RES, F.Cu at (146.7, 114.9)
- added R4: 4k7, SPCoast:0603-RES, F.Cu at (142.9, 114.9)
- added R5: 10k0, SPCoast:0603-RES, F.Cu at (177.0, 111.3)
- added R6: 10k0, SPCoast:0603-RES, F.Cu at (178.9, 111.3)
- added R7: 10k0, SPCoast:0603-RES, F.Cu at (180.8, 111.3)
- added R8: 220R, SPCoast:0603-RES, F.Cu at (203.8, 100.2)
- added R9: 220R, SPCoast:0603-RES, F.Cu at (203.8, 102.1)
- added SJ1: OFF, Jumper:SolderJumper-2_P1.3mm_Bridged_RoundedPad1.0x1.5mm, F.Cu at (186.7, 76.3)
- added SJ10: OFF, Jumper:SolderJumper-2_P1.3mm_Bridged_RoundedPad1.0x1.5mm, F.Cu at (220.3, 76.3)
- added SJ11: OFF, Jumper:SolderJumper-2_P1.3mm_Bridged_RoundedPad1.0x1.5mm, F.Cu at (217.8, 76.3)
- added SJ12: OFF, Jumper:SolderJumper-2_P1.3mm_Bridged_RoundedPad1.0x1.5mm, F.Cu at (215.3, 76.3)
- added SJ13: OFF, Jumper:SolderJumper-2_P1.3mm_Bridged_RoundedPad1.0x1.5mm, F.Cu at (212.7, 76.3)
- added SJ14: OFF, Jumper:SolderJumper-2_P1.3mm_Bridged_RoundedPad1.0x1.5mm, F.Cu at (210.2, 76.3)
- added SJ15: OFF, Jumper:SolderJumper-2_P1.3mm_Bridged_RoundedPad1.0x1.5mm, F.Cu at (207.6, 76.2)
- added SJ16: OFF, Jumper:SolderJumper-2_P1.3mm_Bridged_RoundedPad1.0x1.5mm, F.Cu at (205.1, 76.2)
- added SJ2: OFF, Jumper:SolderJumper-2_P1.3mm_Bridged_RoundedPad1.0x1.5mm, F.Cu at (184.2, 76.3)
- added SJ3: OFF, Jumper:SolderJumper-2_P1.3mm_Bridged_RoundedPad1.0x1.5mm, F.Cu at (181.6, 76.3)
- added SJ4: OFF, Jumper:SolderJumper-2_P1.3mm_Bridged_RoundedPad1.0x1.5mm, F.Cu at (179.1, 76.3)
- added SJ5: OFF, Jumper:SolderJumper-2_P1.3mm_Bridged_RoundedPad1.0x1.5mm, F.Cu at (176.5, 76.3)
- added SJ6: OFF, Jumper:SolderJumper-2_P1.3mm_Bridged_RoundedPad1.0x1.5mm, F.Cu at (174.0, 76.3)
- added SJ7: OFF, Jumper:SolderJumper-2_P1.3mm_Bridged_RoundedPad1.0x1.5mm, F.Cu at (171.4, 76.3)
- added SJ8: OFF, Jumper:SolderJumper-2_P1.3mm_Bridged_RoundedPad1.0x1.5mm, F.Cu at (168.9, 76.3)
- added SJ9: OFF, Jumper:SolderJumper-2_P1.3mm_Bridged_RoundedPad1.0x1.5mm, F.Cu at (222.9, 76.3)
- added SW1: ~, SPCoast:SW-EDG-04, F.Cu at (188.6, 114.9)
- added U1: MCP23017_SO, Package_SO:SOIC-28W_7.5x17.9mm_P1.27mm, F.Cu at (182.2, 95.2)
- added U2: 74HC4511D,653, Package_SO:SOIC-16_3.9x9.9mm_P1.27mm, F.Cu at (196.2, 102.2)
- added U3: ARKLED SM420561N, Display_7Segment:D1X8K, F.Cu at (208.9, 111.0)
- added VR1: LM78M05_TO252-2, Package_TO_SOT_SMD:TO-252-2, F.Cu at (147.3, 79.4)
Routing:
- net +5V: track 0.00 -> 291.5 mm, vias 0 -> 3
- net +VDC: track 0.00 -> 226.3 mm
- net SDA: track 0.00 -> 221.4 mm, vias 0 -> 4
- net SCL: track 0.00 -> 210.2 mm, vias 0 -> 4
- net Net-(J18-Pin_1): track 0.00 -> 46.5 mm
- net Net-(J18-Pin_2): track 0.00 -> 43.4 mm
- net Net-(J18-Pin_3): track 0.00 -> 40.3 mm
- net /A2: track 0.00 -> 37.8 mm, vias 0 -> 5
- net Net-(J18-Pin_4): track 0.00 -> 37.3 mm
- net /A1: track 0.00 -> 37.1 mm, vias 0 -> 4
- net GND: track 0.00 -> 37.0 mm, vias 0 -> 34
- net Net-(J18-Pin_5): track 0.00 -> 34.2 mm
- net Net-(J18-Pin_6): track 0.00 -> 31.1 mm
- net Net-(J14-Pin_8): track 0.00 -> 29.5 mm
- net /A0: track 0.00 -> 29.3 mm, vias 0 -> 2
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- added copper zone on B.Cu, net GND
- added copper zone on F.Cu, net GND
Other:
- board outline added: 110 x 68.5 mm
- copper layers 0 -> 2
- board text added: "${PROJECTNAME}"
- board text added: "-nc-"
- board text added: "0x2"
- board text added: "1"
- board text added: "1 0"
- board text added: "10"
- board text added: "11"
- board text added: "12"
- board text added: "13"
- board text added: "14"
- board text added: "15"
- board text added: "16"
- board text added: "16 bit I2C Expander"
- board text added: "2"
- board text added: "3"
- board text added: "4"
- board text added: "5"
- board text added: "5v"
- board text added: "6"
- board text added: "7"
- board text added: "8"
- board text added: "9"
- board text added: "A0"
- board text added: "A1"
- board text added: "A2"
- board text added: "GND"
- board text added: "I2C Address"
- board text added: "Port A"
- board text added: "Port B"
- board text added: "Power Reversed Good"
- board text added: "V+"
